Commit message: some_changes

File: hector_quadrotor/hector_quadrotor_description/urdf/quadrotor_hokuyo_utm30lx.urdf.xacro (robot description, xacro)
@@ -1,4 +1,6 @@
 <?xml version="1.0"?>
 <robot name="quadrotor" xmlns:xacro="http://www.ros.org/wiki/xacro">
+    <xacro:arg name="gpu" default="false"/>
+    <xacro:property name="gpu" value="$(arg gpu)" />
     <xacro:property name="M_PI" value="3.1415926535897931" />
     <!-- Included URDF Files -->
@@ -12,7 +14,20 @@
     </xacro:hokuyo_utm30lx>
     <!-- Forward facing camera -->
-    <xacro:include filename="$(find hector_sensors_description)/urdf/generic_camera.urdf.xacro" />
+    <!-- <xacro:include filename="$(find hector_sensors_description)/urdf/generic_camera.urdf.xacro" />
     <xacro:generic_camera name="front_cam" parent="base_link" ros_topic="camera/image" cam_info_topic="camera/camera_info" update_rate="30" res_x="640" res_y="480" image_format="R8G8B8" hfov="90">
       <origin xyz="0.05 -0.0 -0.25" rpy="0 0 0"/>
-    </xacro:generic_camera>
+    </xacro:generic_camera> -->
+    <xacro:include filename="$(find hector_sensors_description)/urdf/asus_camera.urdf.xacro" />
+    <xacro:asus_camera name="camera" parent="base_link">
+      <origin xyz="0.0 0.0 -0.097" rpy="${M_PI} 0 0"/>
+    </xacro:asus_camera>
+  <xacro:include filename="/home/dimitris/DRL-robot-navigation/catkin_ws/src/velodyne_simulator/velodyne_description/urdf/VLP-16.urdf.xacro" />
+  <xacro:VLP-16 parent="base_link" name="velodyne" topic="/velodyne_points"  hz="10" samples="440" gpu="True">
+        <origin xyz="0.0 0.0 -0.097" rpy="0 0 0"/>
+    <!-- Adjust vertical FOV to scan directly underneath -->
+  </xacro:VLP-16>
+    <!-- <xacro:include filename="/home/dimitris/DRL-robot-navigation/catkin_ws/src/velodyne_simulator/velodyne_description/urdf/HDL-32E.urdf.xacro"/>
+  <xacro:HDL-32E parent="base_link" name="velodyne2" topic="/velodyne_points2" hz="10" samples="220" gpu="${gpu}">
+    <origin xyz="0 0 0.6" rpy="0 0 0" />
+  </xacro:HDL-32E> -->
 </robot>
