Commit message: happy

File: hector_models/hector_sensors_description/urdf/asus_camera.urdf.xacro (robot description, xacro)
@@ -75,15 +75,16 @@
       <gazebo reference="${name}_depth_frame">
         <sensor type="depth" name="${name}">
-          <update_rate>20</update_rate>
+          <update_rate>30</update_rate>
           <camera>
-            <horizontal_fov>${62.8 * M_PI/180.0}</horizontal_fov>
+            <horizontal_fov>${122.8 * M_PI/180.0}</horizontal_fov>
+            <!-- <horizontal_fov>${62.8 * M_PI/180.0}</horizontal_fov> -->
             <image>
               <format>R8G8B8</format>
-              <width>640</width>
-              <height>480</height>
+              <width>1280</width>
+              <height>720</height>
             </image>
             <clip>
               <near>0.5</near>
-              <far>9</far>
+              <far>50</far>
             </clip>
           </camera>

File: hector_quadrotor/hector_quadrotor_description/urdf/quadrotor_hokuyo_utm30lx.urdf.xacro (robot description, xacro)
@@ -9,22 +9,31 @@
     <xacro:quadrotor_base_macro />
     <!-- Hokuyo UTM-30LX mounted upside down below the quadrotor body -->
-    <xacro:include filename="$(find hector_sensors_description)/urdf/hokuyo_utm30lx.urdf.xacro" />
+    <!-- <xacro:include filename="$(find hector_sensors_description)/urdf/hokuyo_utm30lx.urdf.xacro" />
     <xacro:hokuyo_utm30lx name="laser0" parent="base_link" ros_topic="scan" update_rate="40" ray_count="1081" min_angle="-135" max_angle="135">
       <origin xyz="0.0 0.0 -0.097" rpy="${M_PI} 0 0"/>
+    </xacro:hokuyo_utm30lx> -->
+      <xacro:include filename="$(find hector_sensors_description)/urdf/hokuyo_utm30lx.urdf.xacro" />
+    <xacro:hokuyo_utm30lx name="laser0" parent="base_link" ros_topic="scan" update_rate="40" ray_count="1081" min_angle="-135" max_angle="135">
+      <origin xyz="0.0 0.0 0.1" rpy="${M_PI} 0 0"/>
     </xacro:hokuyo_utm30lx>
     <!-- Forward facing camera -->
-    <!-- <xacro:include filename="$(find hector_sensors_description)/urdf/generic_camera.urdf.xacro" />
-    <xacro:generic_camera name="front_cam" parent="base_link" ros_topic="camera/image" cam_info_topic="camera/camera_info" update_rate="30" res_x="640" res_y="480" image_format="R8G8B8" hfov="90">
+    <xacro:include filename="$(find hector_sensors_description)/urdf/generic_camera.urdf.xacro" />
+    <xacro:generic_camera name="front_cam" parent="base_link" ros_topic="camera/image" cam_info_topic="camera/camera_info" update_rate="30" res_x="160" res_y="120" image_format="R8G8B8" hfov="90">
       <origin xyz="0.05 -0.0 -0.25" rpy="0 0 0"/>
-    </xacro:generic_camera> -->
+    </xacro:generic_camera>
     <xacro:include filename="$(find hector_sensors_description)/urdf/asus_camera.urdf.xacro" />
     <xacro:asus_camera name="camera" parent="base_link">
-      <origin xyz="0.0 0.0 -0.097" rpy="${M_PI} 0 0"/>
+      <!-- <origin xyz="0.0 0.0 -0.097" rpy="${M_PI} 0 0"/> -->
+      <origin xyz="0.0 0.0 -0.097" rpy="0 -0.7 0"/>
     </xacro:asus_camera>
-  <xacro:include filename="/home/dimitris/DRL-robot-navigation/catkin_ws/src/velodyne_simulator/velodyne_description/urdf/VLP-16.urdf.xacro" />
+    <!-- big fov -->
+    <!-- <xacro:include filename="$(find hector_sensors_description)/urdf/asus_camera.urdf.xacro" />
+    <xacro:asus_camera name="camera" parent="base_link">
+      <origin xyz="0.0 0.0 -0.097" rpy="0 -0.7 0"/>
+    </xacro:asus_camera> -->
+  <!-- <xacro:include filename="/home/dimitris/DRL-robot-navigation/catkin_ws/src/velodyne_simulator/velodyne_description/urdf/VLP-16.urdf.xacro" />
   <xacro:VLP-16 parent="base_link" name="velodyne" topic="/velodyne_points"  hz="10" samples="440" gpu="True">
-        <origin xyz="0.0 0.0 -0.097" rpy="0 0 0"/>
-    <!-- Adjust vertical FOV to scan directly underneath -->
-  </xacro:VLP-16>
+        <origin xyz="0.0 0.0 -0.097" rpy="${M_PI} 0 0"/>
+  </xacro:VLP-16> -->
     <!-- <xacro:include filename="/home/dimitris/DRL-robot-navigation/catkin_ws/src/velodyne_simulator/velodyne_description/urdf/HDL-32E.urdf.xacro"/>
   <xacro:HDL-32E parent="base_link" name="velodyne2" topic="/velodyne_points2" hz="10" samples="220" gpu="${gpu}">
